File: PCB/Lora Tester (EEPROM Programmer).kicad_sch (KiCad schematic)
At the start: 4 parts, among them J1 Raspberry Pi GPIO Connector, J2 Conn_01x03, U1 ZIF Socket, U2 24C01-24C1024

Commit message: all done
Parts:
- J1: symbol pi-eeprom-programmer-rescue:Conn_02x20_Odd_Even-Connector_Generic -> Lora Tester-rescue:Conn_02x20_Odd_Even-Connector_Generic
- U1: symbol pi-eeprom-programmer-rescue:28C256-Memory_EEPROM -> Lora Tester-rescue:28C256-Memory_EEPROM
Changed lines of the file:
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@@
 	)
 	(symbol
-		(lib_id "pi-eeprom-programmer-rescue:Conn_02x20_Odd_Even-Connector_Generic")
+		(lib_id "Lora Tester-rescue:Conn_02x20_Odd_Even-Connector_Generic")
 		(at 73.66 67.31 0)
 		(unit 1)
@@
 	)
 	(symbol
-		(lib_id "pi-eeprom-programmer-rescue:28C256-Memory_EEPROM")
+		(lib_id "Lora Tester-rescue:28C256-Memory_EEPROM")
 		(at 200.66 63.5 0)
 		(unit 1)
